Commit message: [fix] fk and fd tree

File: examples/urdf/alpha_5_robot_for_FK.urdf (robot description, URDF)
Before this commit: robot alpha_5_example, 12 links, 11 joints
Joints:
- joint alpha_axis_c: axis 0 -1 0 -> 0 1 0; limit lower=-3.5 upper=0.0 effort=9.0 velocity=0.5 -> lower=0.2 upper=3.4 effort=9.0 velocity=0.5
