Commit message: added meshes

File: usage/urdf/reach_alpha_5/alpha_5_robot.urdf (robot description, URDF)
Before this commit: robot alpha_5_example, 12 links, 11 joints
Links:
- link alpha_m1_link: geometry collision cylinder length=0.10975 radius=0.020; visual mesh filename=./meshes/RS1-100-101-123.stl
- link alpha_m2_1_1_link: geometry collision cylinder length=0.066 radius=0.020; visual mesh filename=./meshes/M2-1-1.stl
- link alpha_m2_1_2_link: geometry collision cylinder length=0.033 radius=0.020; visual mesh filename=./meshes/M2-1-3.stl
- link alpha_m2_joint_link: geometry collision cylinder length=0.040 radius=0.020; collision cylinder length=0.040 radius=0.020
- link alpha_m3_inline_link: geometry collision cylinder length=0.100 radius=0.020; visual mesh filename=./meshes/M3-INLINE.stl
- link alpha_standard_jaws_base_link: geometry visual mesh filename=./meshes/end_effectors/RS1-124.stl
- link alpha_standard_jaws_rs1_130_link: geometry collision box size=0.012 0.03 0.09; visual mesh filename=./meshes/end_effectors/RS1-130.stl
- link alpha_standard_jaws_rs1_139_link: geometry collision box size=0.012 0.03 0.09; visual mesh filename=./meshes/end_effectors/RS1-139.stl
